Commit message: Correctamente medido con guillermo

File: urdf/robot2.urdf (robot description, URDF)
Before this commit: robot robot2, 11 links, 10 joints
Links:
- link base_batteries: geometry collision box size=0.3031 0.065 0.0939; visual box size=0.3031 0.065 0.0939
- link base_link: geometry collision box size=0.4231 0.25158 0.0515; visual box size=0.4231 0.25158 0.0515
- link base_wifi: geometry collision box size=0.0275 0.1857 0.1202; visual box size=0.0275 0.1857 0.1202
- link left_back_motor: geometry collision cylinder length=0.0439 radius=0.023; visual cylinder length=0.0439 radius=0.023
- link left_back_wheel: geometry collision cylinder length=0.077 radius=0.1295; visual cylinder length=0.077 radius=0.1295
- link left_front_motor: geometry collision cylinder length=0.0439 radius=0.023; visual cylinder length=0.0439 radius=0.023
- link left_front_wheel: geometry collision cylinder length=0.077 radius=0.1295; visual cylinder length=0.077 radius=0.1295
- link right_back_motor: geometry collision cylinder length=0.0439 radius=0.023; visual cylinder length=0.0439 radius=0.023
- link right_back_wheel: geometry collision cylinder length=0.077 radius=0.1295; visual cylinder length=0.077 radius=0.1295
- link right_front_motor: geometry collision cylinder length=0.0439 radius=0.023; visual cylinder length=0.0439 radius=0.023
- link right_front_wheel: geometry collision cylinder length=0.077 radius=0.1295; visual cylinder length=0.077 radius=0.1295
Joints:
- joint base_to_wifi: origin xyz=-0.3 0 0 -> xyz=-0.2253 0 0
- joint left_back_motor_joint: origin xyz=-0.27 0.275 0 rpy=0 0 0 -> xyz=-0.18855 0.12579 0 rpy=0 0 0
- joint left_back_wheel_joint: origin xyz=0.0 0.075 0 rpy=0 0 0 -> xyz=0.0 0.06045 0 rpy=0 0 0
- joint left_front_motor_joint: origin xyz=0.27 0.275 0 rpy=0 0 0 -> xyz=0.18855 0.12579 0 rpy=0 0 0
- joint left_front_wheel_joint: origin xyz=0.0 0.075 0 rpy=0 0 0 -> xyz=0.0 0.06045 0 rpy=0 0 0
- joint right_back_motor_joint: origin xyz=-0.27 -0.275 0 rpy=0 0 0 -> xyz=-0.18855 -0.12579 0 rpy=0 0 0
- joint right_back_wheel_joint: origin xyz=0.0 -0.075 0 rpy=0 0 0 -> xyz=0.0 -0.06045 0 rpy=0 0 0
- joint right_front_motor_joint: origin xyz=0.27 -0.275 0 rpy=0 0 0 -> xyz=0.18855 -0.12579 0 rpy=0 0 0
- joint right_front_wheel_joint: origin xyz=0.0 -0.075 0 rpy=0 0 0 -> xyz=0.0 -0.06045 0 rpy=0 0 0
